File: PCB/DynaLab/DynaLab.kicad_sch (KiCad schematic)
At the start: 96 parts, among them J1 USB_C_Receptacle_USB2.0_16P, SW1 BOOT, SW2 REC/STOP, SW3 RESET, U1 LM393, U10 74AHCT125, U11 ITR8307-S17-TR8, U12 ITR8307-S17-TR8, U13 USBLC6-2SC6, U14 RP2040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

Commit message: atomise PCB projects for portability
Parts:
- removed D1: REC, LED_SMD:LED_0603_1608Metric, symbol Device:LED
- removed R26: 220, Resistor_SMD:R_0603_1608Metric, symbol Device:R
- D2: LCSC Part # C965804 -> C965807
- H1, H2, H3, H4, H5, H6, H7, H8: value SMTSO3030 -> SMTSO3060; footprint Footprints:MountingHole_SMTSO3030_3.2mm_M3 -> Footprints:MountingHole_SMTSO3060_3.2mm_M3; LCSC Part # C2915308 -> C2915637
- H10, H11, H12, H9: value SMTSO3040 -> SMTSO3080; footprint Footprints:MountingHole_SMTSO3030_3.2mm_M3 -> Footprints:MountingHole_SMTSO3080_3.2mm_M3; LCSC Part # C2915635 -> C2916369
- R30: value 1k -> 220
- SW2: footprint Button_Switch_THT:SW_PUSH-12mm -> Button_Switch_THT:SW_SPST_Omron_B3F-40xx; LCSC Part # C5381278 -> C84931
- SW3: footprint Button_Switch_THT:SW_PUSH-12mm -> Button_Switch_THT:SW_SPST_Omron_B3F-40xx; LCSC Part # C7470193 -> C84931
- U5, U6, U7: symbol Display_Character:SM420561N -> DynaLab_Symbols:GS3011C
Connections:
- net GND: now also SW1.2; no longer SW1.1
- net ~{BOOT}: now also SW1.1; no longer SW1.2
- net LED_REC: no longer names the net of U14.36 (GPIO24)
- no-connect marks 34 -> 35
Other:
- note added: "M3x6mm"
- note added: "M3x8mm"
- note added: "SMT Solder in-place"
- note added: "Threaded Standoffs"
- note added: "USB-C spec calls for 5k1 (10%) pulldown resistors on CC1, CC2 10k || 10k = 5k (1%) should work - optimise BOM"
- note removed: "M3x3mm threaded standoffs"
- note removed: "M3x4mm threaded standoffs"
- moved on the sheet: H1, H10, H11, H12, H2, H3, H4, H5, H6, H7, H8, H9

Commit message: add purchasing #s and some datasheets
Parts:
- C1, C2, C21, C22, C3, C4: value 100n -> 100nF
- C14, C15: LCSC Part # (none) -> C15849
- C17, C18: LCSC Part # (none) -> C1656
- C19, C20: LCSC Part # (none) -> C19702
- R1, R25, R27, R4: LCSC Part # (none) -> C21190
- R10, R11, R12, R15, R16, R17, R2, R20, R21, R22, R28, R29, R3, R31, R32, R5, R7, R9: LCSC Part # (none) -> C25804
- R13, R18, R6: LCSC Part # (none) -> C22807
- R14, R19, R30, R8: LCSC Part # (none) -> C22962
- R23, R24: LCSC Part # (none) -> C25190
Other:
- note added: "ERC Suppress power-related errors"
